Commit message: Use sim2sim G1 head URDF

File: holosoma_robot_description/urdf/g1_29dof.urdf (robot description, URDF)
Before this commit: robot g1, 42 links, 41 joints
Links:
- added link mid360_link_IMU; visual box size=0.001 0.001 0.001
- added link mid360_link_frame; visual box size=0.001 0.001 0.001
- link left_rubber_hand: geometry visual mesh filename=package://holosoma_robot_description/urdf/meshes/left_rubbe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
- link left_wrist_yaw_link: geometry collision cylinder length=0.05 radius=0.05; visual mesh filename=package://holosoma_robot_description/urdf/meshes/left_wrist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
- link right_rubber_hand: geometry visual mesh filename=package://holosoma_robot_description/urdf/meshes/right_rubb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
- link right_wrist_yaw_link: geometry collision cylinder length=0.05 radius=0.05; visual mesh filename=package://holosoma_robot_description/urdf/meshes/right_wris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
Joints:
- added joint mid360_frame_joint: type fixed, parent mid360_link, child mid360_link_frame, origin xyz=0 0 0 rpy=3.14159 0 0
- added joint mid360_imu_joint: type fixed, parent mid360_link_frame, child mid360_link_IMU, origin xyz=0.011 0.02329 -0.04412 rpy=0 0 0
- joint head_joint: origin xyz=0.0039635 0 -0.044 rpy=0 0 0 -> xyz=0.015 0 0.43 rpy=0 0 0
- joint mid360_joint: origin xyz=0.0002835 0.00003 0.41618 rpy=0 3.101 3.1415 -> xyz=0.0002835 0.00003 0.41618 rpy=0 0.04014257279586953 0
